File: hardware/v02/02.brd (EAGLE design)
At the start: 79.7 x 38.1 mm, 29 parts, among them IC2 78L05Z, IC3 MSP430G2553, X2 RJ45-6L-B

Commit message: minor changes
Parts:
- C3: value 100nF -> 2.2nF
Changed lines of the file:
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@@
 </element>
 <element name="R10" library="rcl" package="0207/7" value="47k" x="73.66" y="19.05" rot="R180"/>
-<element name="C3" library="rcl" package="C025-024X044" value="100nF" x="66.04" y="17.78" rot="R270"/>
+<element name="C3" library="rcl" package="C025-024X044" value="2.2nF" x="66.04" y="17.78" rot="R270"/>
 <element name="RN1" library="resistor-net" package="RN-5" value="4.7k" x="11.43" y="19.05">
 <attribute name="OC_NEWARK" value="unknown" x="11.43" y="19.05" size="1.778" layer="27" display="off"/>
