File: hardware/v02/02.sch (EAGLE design)
At the start: 29 parts, among them IC2 78L05Z, IC3 MSP430G2553, X2 RJ45-6L-B

Commit message: minor changes
Parts:
- C3: value 100nF -> 2.2nF
Changed lines of the file:
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@@
 <part name="GND4" library="supply1" deviceset="GND" device=""/>
 <part name="R10" library="rcl" deviceset="R-EU_" device="0207/7" value="47k"/>
-<part name="C3" library="rcl" deviceset="C-EU" device="025-024X044" value="100nF"/>
+<part name="C3" library="rcl" deviceset="C-EU" device="025-024X044" value="2.2nF"/>
 <part name="P+10" library="supply1" deviceset="VCC" device=""/>
 <part name="FRAME1" library="frames" deviceset="DINA5_L" device=""/>

Commit message: echange pin header; labels on top
Parts:
- JP5: device pinhead:PINHD-1X4/90 -> pinhead:PINHD-1X4
Changed lines of the file:
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@@
 <part name="JP3" library="pinhead" deviceset="PINHD-1X3" device=""/>
 <part name="JP4" library="pinhead" deviceset="PINHD-1X3" device=""/>
-<part name="JP5" library="pinhead" deviceset="PINHD-1X4" device="/90"/>
+<part name="JP5" library="pinhead" deviceset="PINHD-1X4" device=""/>
 <part name="X2" library="con-tycoelectronics" deviceset="RJ45" device="" technology="-6L-B"/>
 <part name="P+8" library="supply1" deviceset="+5V" device=""/>
